File: PCIe_x16-to-x8_Debifurcator.kicad_pcb (KiCad board)
At the start: 4 copper layers, 28.5 x 85.6 mm, 7 parts, among them J1 PCI_Express_x8, J2 PCI_Express_x16

Commit message: v0.1.1 PCB Layout Updated
Parts:
- added C1: 0u1, Capacitor_SMD:C_0603_1608Metric_Pad1.08x0.95mm_HandSolder, F.Cu at (81.1, 59.9)
- moved TP3 0.40 mm to (80.0, 82.6)
Routing:
- net GND: track 999.9 -> 815.1 mm, vias 75 -> 122
- net Tx1_P: track 59.5 -> 65.2 mm
- net Tx3_N: track 59.5 -> 62.9 mm
- net Rx1_N: track 58.8 -> 62.0 mm
- net Tx3_P: track 59.7 -> 63.0 mm
- net Tx1_N: track 59.5 -> 62.6 mm
- net Tx7_N: track 58.9 -> 61.9 mm
- net Rx1_P: track 59.0 -> 62.0 mm
- net Tx0_N: track 59.6 -> 61.9 mm
- net Rx0_P: track 59.7 -> 62.0 mm
- net Rx2_P: track 59.8 -> 62.0 mm
- net Tx6_P: track 60.1 -> 61.9 mm
- net Rx2_N: track 58.5 -> 60.1 mm
- net /PRSNT1: track 180.8 -> 182.3 mm
- net Tx5_P: track 60.1 -> 61.5 mm
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