File: PCIe_x16-to-x8_Debifurcator.kicad_sch (KiCad schematic)
At the start: 7 parts, among them J1 PCI_Express_x8, J2 PCI_Express_x16

Commit message: v0.1.1 PCB Layout Updated
Parts:
- added C1: 0u1, Capacitor_SMD:C_0603_1608Metric_Pad1.08x0.95mm_HandSolder, symbol Device:C_Small
Connections:
- net GND: now also C1.2
- net PRSNT1: now also C1.1
Changed lines of the file:
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@@
+    (stroke (width 0) (type default))
+  )
+  (wire (pts (xy 20.32 46.99) (xy 20.32 48.26))
     (stroke (width 0) (type default))
   )
@@
     (stroke (width 0) (type default))
   )
+  (wire (pts (xy 20.32 40.64) (xy 20.32 41.91))
+    (stroke (width 0) (type default))
+  )
+  (label "PRSNT1" (at 20.32 40.64 180) (fields_autoplaced)
+    (effects (font (size 1.27 1.27)) (justify right bottom))
+  )
   (label "PRSNT1" (at 99.06 63.5 180) (fields_autoplaced)
     (effects (font (size 1.27 1.27)) (justify right bottom))
@@
   )
   (symbol (lib_id "power:GND") (at 55.88 120.65 0) (unit 1)
+    (in_bom yes) (on_board yes) (dnp no)
+    (property "Reference" "#PWR0101" (at 55.88 127 0)
+      (effects (font (size 1.27 1.27)) hide)
+    )
+    (property "Value" "GND" (at 55.88 124.46 0)
+      (effects (font (size 1.27 1.27)))
+    )
+    (property "Footprint" "" (at 55.88 120.65 0)
+      (effects (font (size 1.27 1.27)) hide)
+    )
+    (property "Datasheet" "" (at 55.88 120.65 0)
+      (effects (font (size 1.27 1.27)) hide)
+    )
+    (pin "1")
+    (instances
+      (project "PCIe_x16-to-x8_Debifurcator"
+        (path "/81468c52-672d-42a3-92d2-29a7c075d013"
+          (reference "#PWR0101") (unit 1)
+        )
+      )
+    )
+  )
+  (symbol (lib_id "Device:C_Small") (at 20.32 44.45 0) (unit 1)
     (in_bom yes) (on_board yes) (dnp no) (fields_autoplaced)
-    (property "Reference" "#PWR0101" (at 55.88 127 0)
-      (effects (font (size 1.27 1.27)) hide)
-    )
-    (property "Value" "GND" (at 55.88 125.73 0)
-      (effects (font (size 1.27 1.27)))
-    )
-    (property "Footprint" "" (at 55.88 120.65 0)
-      (effects (font (size 1.27 1.27)) hide)
-    )
-    (property "Datasheet" "" (at 55.88 120.65 0)
-      (effects (font (size 1.27 1.27)) hide)
-    )
-    (pin "1")
-    (instances
-      (project "PCIe_x16-to-x8_Debifurcator"
-        (path "/81468c52-672d-42a3-92d2-29a7c075d013"
-          (reference "#PWR0101") (unit 1)
+    (property "Reference" "C1" (at 22.86 43.1863 0)
+      (effects (font (size 1.27 1.27)) (justify left))
+    )
+    (property "Value" "0u1" (at 22.86 45.7263 0)
+      (effects (font (size 1.27 1.27)) (justify left))
+    )
+    (property "Footprint" "Capacitor_SMD:C_0603_1608Metric_Pad1.08x0.95mm_HandSolder" (at 20.32 44.45 0)
+      (effects (font (size 1.27 1.27)) hide)
+    )
+    (property "Datasheet" "~" (at 20.32 44.45 0)
+      (effects (font (size 1.27 1.27)) hide)
+    )
+    (pin "1")
+    (pin "2")
+    (instances
+      (project "PCIe_x16-to-x8_Debifurcator"
+        (path "/81468c52-672d-42a3-92d2-29a7c075d013"
+          (reference "C1") (unit 1)
         )
       )
@@
   )
   (symbol (lib_id "power:GND") (at 114.3 166.37 0) (unit 1)
-    (in_bom yes) (on_board yes) (dnp no) (fields_autoplaced)
+    (in_bom yes) (on_board yes) (dnp no)
     (property "Reference" "#PWR06" (at 114.3 172.72 0)
       (effects (font (size 1.27 1.27)) hide)
     )
-    (property "Value" "GND" (at 114.3 171.45 0)
+    (property "Value" "GND" (at 114.3 170.18 0)
       (effects (font (size 1.27 1.27)))
     )
@@
         )
       )
+    )
+  )
+  (symbol (lib_id "power:GND") (at 20.32 48.26 0) (unit 1)
+    (in_bom yes) (on_board yes) (dnp no)
+    (property "Reference" "#PWR08" (at 20.32 54.61 0)
+      (effects (font (size 1.27 1.27)) hide)
+    )
+    (property "Value" "GND" (at 20.32 52.07 0)
+      (effects (font (size 1.27 1.27)))
+    )
+    (property "Footprint" "" (at 20.32 48.26 0)
+      (effects (font (size 1.27 1.27)) hide)
+    )
+    (property "Datasheet" "" (at 20.32 48.26 0)
+      (effects (font (size 1.27 1.27)) hide)
+    )
+    (pin "1")
+    (instances
+      (project "PCIe_x16-to-x8_Debifurcator"
+        (path "/81468c52-672d-42a3-92d2-29a7c075d013"
+          (reference "#PWR08") (unit 1)
+        )
+      )
